File: boris-board.kicad_pcb (KiCad board)
At the start: 4 copper layers, 35 x 55 mm, 24 parts

Commit message: Add some stuff
Signed-off-by: Michael Welling <mwelling@ieee.org>
Parts:
- removed REF** (x20): SK6805-2427, PocketBeagle.pretty:SK6805-2427
- added LD1: SK6805-2427, PocketBeagle.pretty:SK6805-2427, F.Cu at (171.7, 137.7)
- added LD10: SK6805-2427, PocketBeagle.pretty:SK6805-2427, F.Cu at (171.7, 101.1)
- added LD11: SK6805-2427, PocketBeagle.pretty:SK6805-2427, F.Cu at (140.0, 101.1)
- added LD12: SK6805-2427, PocketBeagle.pretty:SK6805-2427, F.Cu at (140.0, 105.2)
- added LD13: SK6805-2427, PocketBeagle.pretty:SK6805-2427, F.Cu at (140.0, 109.2)
- added LD14: SK6805-2427, PocketBeagle.pretty:SK6805-2427, F.Cu at (140.0, 113.3)
- added LD15: SK6805-2427, PocketBeagle.pretty:SK6805-2427, F.Cu at (140.0, 117.3)
- added LD16: SK6805-2427, PocketBeagle.pretty:SK6805-2427, F.Cu at (140.0, 121.4)
- added LD17: SK6805-2427, PocketBeagle.pretty:SK6805-2427, F.Cu at (140.0, 125.5)
- added LD18: SK6805-2427, PocketBeagle.pretty:SK6805-2427, F.Cu at (140.0, 129.5)
- added LD19: SK6805-2427, PocketBeagle.pretty:SK6805-2427, F.Cu at (140.0, 133.6)
- added LD2: SK6805-2427, PocketBeagle.pretty:SK6805-2427, F.Cu at (171.7, 133.6)
- added LD20: SK6805-2427, PocketBeagle.pretty:SK6805-2427, F.Cu at (140.0, 138.2)
- added LD3: SK6805-2427, PocketBeagle.pretty:SK6805-2427, F.Cu at (171.7, 129.5)
- added LD4: SK6805-2427, PocketBeagle.pretty:SK6805-2427, F.Cu at (171.7, 125.5)
- added LD5: SK6805-2427, PocketBeagle.pretty:SK6805-2427, F.Cu at (171.7, 121.4)
- added LD6: SK6805-2427, PocketBeagle.pretty:SK6805-2427, F.Cu at (171.7, 117.3)
- added LD7: SK6805-2427, PocketBeagle.pretty:SK6805-2427, F.Cu at (171.7, 113.3)
- added LD8: SK6805-2427, PocketBeagle.pretty:SK6805-2427, F.Cu at (171.7, 109.2)
- added LD9: SK6805-2427, PocketBeagle.pretty:SK6805-2427, F.Cu at (171.7, 105.2)
- LOGO1: footprint boris-board:boris -> PocketBeagle.pretty:boris
- P1, P2: footprint boris-board:SMT-HEADER-HACK -> PocketBeagle.pretty:SMT-HEADER-HACK
- moved LOGO2 24.3 mm to (155.7, 142.2)
- moved LOGO1 6.07 mm to (155.8, 119.4)
Connections:
- P1 pad 14: VDD_3V3B -> Net-(P1-Pad14)
Routing:
- net SYS_5V: track 0.00 -> 159.2 mm, vias 0 -> 2
- net GND: track 0.00 -> 84.6 mm, vias 0 -> 2
- net Net-(LD10-Pad1): track 0.00 -> 34.7 mm, vias 0 -> 2
- net /(U1.A2)PRU-0.1: track 0.00 -> 3.76 mm, vias 0 -> 1
- net Net-(LD19-Pad1): track 0.00 -> 3.23 mm
- net Net-(LD2-Pad1): track 0.00 -> 2.72 mm
- net Net-(LD18-Pad1): track 0.00 -> 2.72 mm
- net Net-(LD7-Pad1): track 0.00 -> 2.72 mm
- net Net-(LD5-Pad1): track 0.00 -> 2.72 mm
- net Net-(LD10-Pad3): track 0.00 -> 2.72 mm
- net Net-(LD15-Pad1): track 0.00 -> 2.72 mm
- net Net-(LD13-Pad1): track 0.00 -> 2.72 mm
- net Net-(LD11-Pad1): track 0.00 -> 2.72 mm
- net Net-(LD3-Pad1): track 0.00 -> 2.72 mm
- net Net-(LD16-Pad1): track 0.00 -> 2.72 mm
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- added copper zone on B.Cu, net GND
Other:
- net class Default: clearance 0 -> 0.1524
- rule trace_clearance: 0 -> 0.1524
