File: boris-board.sch (KiCad schematic (older format))
At the start: 4 parts

Commit message: Add some stuff
Signed-off-by: Michael Welling <mwelling@ieee.org>
Parts:
- added LD1, LD10, LD11, LD12, LD13, LD14, LD15, LD16, LD17, LD18, LD19, LD2, LD20, LD3, LD4, LD5, LD6, LD7, LD8, LD9: SK6805-2427, PocketBeagle.pretty:SK6805-2427, symbol SK6805-2427
Connections:
- wire segments 72 -> 175
